Commit message: feat: add camera TF chain for eye-in-hand calibration and 3D point transform
Publish static TF from hand → camera_link → camera_color_optical_frame
via CameraExtrinsics config. Expose transform_to_base() on GraspTaskManager
and add camera TF verification test.

File: urdf/panda.urdf (robot description, URDF)
Before this commit: robot panda, 13 links, 12 joints
Links:
- added link camera_color_optical_frame
- added link camera_link
- link panda_link0: mass 2.9 -> None
Joints:
- added joint camera_color_optical_joint: type fixed, parent camera_link, child camera_color_optical_frame, origin xyz=0 0 0 rpy=-1.57079632679 0 -1.57079632679
- added joint panda_hand_camera_joint: type fixed, parent panda_hand, child camera_link, origin xyz=0.015 0 0.03 rpy=0 1.57079632679 3.14159265359
