Commit message: fix: multi-package improvements for thread safety and UI reliability
- robot_controller: add tcp_to_matrix4d helper, use shared_mutex for RobotState,
  add mutex for IK solver last_result cache, fix gripper publishing to include
  arm joints, replace std::cout with RCLCPP logging, add motion cancellation
- robot_hmi: fix QImage lifetime with .copy(), add Jog button mouse leave handling,
  add jog_mutex_ for thread safety, add emergency_active_ flag for fault recovery
- robot_vision: use atomic for GraspState, add TF lookup validation, remove
  hard-coded sleep delays
- robot_description: fix mesh file paths (collision → visual)
- robot_api_python: add CONTROL_LOOP_HZ constant and velocity_ik binding
- robot_msgs: document frame field in action definitions

File: src/robot_description/urdf/panda.urdf (robot description, URDF)
Before this commit: robot panda, 15 links, 14 joints
Links:
- link panda_link0: geometry collision mesh filename=package://meshes/collision/link0.obj; visual mesh filename=package://meshes/visual/link0.obj
- link panda_link7: geometry collision mesh filename=package://meshes/collision/link7.obj; visual mesh filename=package://meshes/visual/link7.obj

Commit message: fix: correct camera mounting orientation in URDF
修正相机安装姿态 RPY 从 [0, 1.5708, 3.1416] 改为 [0, -1.5708, 0]，
使 camera_link X 轴指向 hand Z 轴负方向（朝下）。

涉及文件：
- robot_description/urdf/panda.urdf: 修改相机 joint 原点姿态
- robot_description/CLAUDE.md: 更新相机参数文档
- robot_controller/.../topic_config.hpp: 同步 CameraExtrinsics rpy 参数

File: src/robot_description/urdf/panda.urdf (robot description, URDF)
Before this commit: robot panda, 15 links, 14 joints
Joints:
- joint panda_hand_camera_joint: origin xyz=0.015 0 0.03 rpy=0 1.57079632679 3.14159265359 -> xyz=0.015 0 0.03 rpy=0 -1.57079632679 0

Commit message: fix(vision): 统一相机外参配置，修正 USD 到 ROS 光学坐标系转换
- robot_description: 更新 URDF 相机位姿（与 Isaac Sim 左目光心一致）
- robot_controller: 修正 TopicConfig 默认外参及 TF 发布（Rx(π) 而非 Ryp(-π/2,0,-π/2)）
- robot_vision: 同步 GraspTaskManager 默认相机参数
- robot_api_python: 更新 pybind11 绑定默认值
- robot_demos: 同步演示代码相机外参

相机外参: xyz=(0.025, -0.015, 0.015), rpy=(π, 0, -π/2)
光学变换: camera_link → optical 为 Rx(π)（USD→ROS 坐标系转换）

File: src/robot_description/urdf/panda.urdf (robot description, URDF)
Before this commit: robot panda, 15 links, 14 joints
Joints:
- joint camera_color_optical_joint: origin xyz=0 0 0 rpy=-1.57079632679 0 -1.57079632679 -> xyz=0 0 0 rpy=3.14159265359 0 0
- joint panda_hand_camera_joint: origin xyz=0.015 0 0.03 rpy=0 -1.57079632679 0 -> xyz=0.025 -0.015 0.015 rpy=3.14159265359 0 -1.57079632679

Commit message: fix(vision): 修正 USD 到 ROS 光学坐标系转换 (Rx→Ry)
将 camera_link → camera_color_optical_frame 的固定旋转变换从
Rx(π) 修正为 Ry(π)，统一所有相关代码和 URDF 定义。

同时增强 HMI 相机面板：点击画面时在控制台输出完整诊断信息，
包括像素坐标、深度、3D 坐标（相机系/基准系）、内参和变换矩阵。

File: src/robot_description/urdf/panda.urdf (robot description, URDF)
Before this commit: robot panda, 15 links, 14 joints
Joints:
- joint camera_color_optical_joint: origin xyz=0 0 0 rpy=3.14159265359 0 0 -> xyz=0 0 0 rpy=0 3.14159265359 0
